Commit message: config moveit and gazebo

File: staubli_description/urdf/tx60l.xacro (robot description, xacro)
@@ -1,5 +1,9 @@
 <?xml version="1.0" ?>
 <robot name="staubli_tx60l" xmlns:xacro="http://wiki.ros.org/xacro">
-  <xacro:include filename="$(find staubli_description)/urdf/tx60l_macro.xacro"/>
-  <xacro:staubli_tx60l prefix=""/>
+  <!--定义prefix属性-->
+  <xacro:property name="prefix" value="" />
+  <!--包含tx60l_macro.xacro文件-->
+  <xacro:include filename="$(find staubli_description)/urdf/tx60l_macro.xacro" />
+  <!--Staubli_tx60l定义-->
+  <xacro:staubli_tx60l prefix="${prefix}" />
 </robot>
